File: lamp.kicad_pcb (KiCad board)
At the start: 4 copper layers, 24 x 24 mm, 47 parts, among them J1 Conn_01x01_Female, J2 Conn_01x01_Female, J3 Conn_01x01_Female, J4 Conn_01x01_Female, J5 Conn_01x01_Female, J6 Conn_01x01_Female, J7 Conn_01x01_Female, U1 STM32F030F4P6, U2 LMV321, U3 MIC5205-3.3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

Commit message: More or less working
Parts:
- moved C14 0.89 mm to (138.4, 87.0)
Routing:
- net /LED2: track 13.6 -> 7.91 mm
- net GND: track 59.4 -> 56.5 mm
- net /LED1: track 11.1 -> 10.1 mm
- net /EN: track 16.8 -> 17.7 mm
